File: 386RC-16.kicad_sch (KiCad schematic)
At the start: 62 parts, among them J1 Bus_ISA_8bit Power only, U1 74HC244, U10 74HC244, U11 74HC244, U12 74HC240, U13 74HC244, U14 74HC240, U15 74HC244, U16 74HC240, U2 74HC244, U3 74HC240, U4 74HC244, U5 74HC240, U6 74LS32, U7 74LS32, U8 74LS32, U9 74LS32

Commit message: Add files via upload
Parts:
- RP1, RP10, RP11, RP12, RP13, RP14, RP15, RP16, RP18, RP19, RP20, RP21, RP23, RP24, RP25, RP26, RP27, RP28: value R_Network07 -> 22 Ohm
- RP17: value 22Ohm -> 22 Ohm
- RP22: value Resistor_THT:R_Array_SIP8 -> 22 Ohm
- U1, U10, U11, U13, U15, U2, U4: value 74HC244 -> 74F244
- U12, U14, U16, U3, U5: value 74HC240 -> 74F240
- U6, U7, U8, U9: value 74LS32 -> 74F32; symbol 74xx:74LS32 -> New_Library:74LS32
Connections:
- net +5V: now also S1.80 (+5V), S1.98 (+5V); no longer S1.78 (+5V), S1.96 (GND)
- net GND: now also S1.78 (GND), S1.96 (GND), SIM1.19 (A10), SIM1.24 (A11), SIM10.19 (A10), SIM10.24 (A11), SIM11.19 (A10), SIM11.24 (A11), SIM12.19 (A10), SIM12.24 (A11), SIM13.19 (A10), SIM13.24 (A11), SIM14.19 (A10), SIM14.24 (A11), SIM15.19 (A10), SIM15.24 (A11), SIM16.19 (A10), SIM16.24 (A11), SIM2.19 (A10), SIM2.24 (A11), SIM3.19 (A10), SIM3.24 (A11), SIM4.19 (A10), SIM4.24 (A11), SIM5.19 (A10), SIM5.24 (A11), SIM6.19 (A10), SIM6.24 (A11), SIM7.19 (A10), SIM7.24 (A11), SIM8.19 (A10), SIM8.24 (A11), SIM9.19 (A10), SIM9.24 (A11); no longer S1.80 (GND), S1.98 (GND)
- no-connect marks 32 -> 0
Other:
- note added: "Power pins on S1 edge connector need verifying against real hardware. Only 31, 62, 80, 98 are correct."
